File: pcb/DSMR-Splitter.kicad_sch (KiCad schematic)
At the start: 56 parts, among them J1 JTAG, J2 UART, J3 IN, J4 OUT-A, J5 OUT-B, J6 OUT-C, U1 EFM32PG12B500, U10 VOH1016AG-V, U11 74AHCT1G04, U12 VOH1016AG-V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

Commit message: Annotate schema with order numbers
Parts:
- C11, C12: Order Number (none) -> Farnell: 2627461
- C2, C4: Order Number (none) -> Farnell: 1833843
- J3, J4, J5, J6: Order Number (none) -> Farnell: 2135977
- U1: Order Number (none) -> DigiKey: 336-3941-ND
- U10, U12, U13, U6, U7, U9: Order Number (none) -> Mouser: 78-VOH1016AB-T
- U11, U4, U5, U8: Order Number (none) -> Farnell: 2057387
- U2: Order Number (none) -> Farnell: 3122539
- U3: Order Number (none) -> Farnell: 3119379
- Y1: Order Number (none) -> DigiKey: 1253-1120-1-ND
Changed lines of the file:
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@@
+      (effects (font (size 1.27 1.27)) hide)
+    )
+    (property "Order Number" "Farnell: 2135977" (id 4) (at 381 39.37 0)
       (effects (font (size 1.27 1.27)) hide)
     )
@@
       (effects (font (size 1.27 1.27)) hide)
     )
+    (property "Order Number" "Farnell: 2135977" (id 4) (at 381 101.6 0)
+      (effects (font (size 1.27 1.27)) hide)
+    )
     (pin "1")
     (pin "2")
@@
       (effects (font (size 1.27 1.27)) hide)
     )
+    (property "Order Number" "Farnell: 2135977" (id 4) (at 381 162.56 0)
+      (effects (font (size 1.27 1.27)) hide)
+    )
     (pin "1")
     (pin "2")
@@
       (effects (font (size 1.27 1.27)) hide)
     )
+    (property "Order Number" "Farnell: 2135977" (id 4) (at 381 222.25 0)
+      (effects (font (size 1.27 1.27)) hide)
+    )
     (pin "1")
     (pin "2")
@@
     )
     (property "Datasheet" "" (id 3) (at 95.25 77.47 0)
+      (effects (font (size 1.27 1.27)) hide)
+    )
+    (property "Order Number" "DigiKey: 336-3941-ND" (id 4) (at 90.17 81.28 0)
       (effects (font (size 1.27 1.27)) hide)
     )
@@
       (effects (font (size 1.27 1.27)) hide)
     )
+    (property "Order Number" "Farnell: 2627461" (id 4) (at 168.91 54.61 0)
+      (effects (font (size 1.27 1.27)) hide)
+    )
     (pin "1")
     (pin "2")
@@
     )
     (property "Datasheet" "~" (id 3) (at 168.91 67.31 0)
+      (effects (font (size 1.27 1.27)) hide)
+    )
+    (property "Order Number" "Farnell: 2627461" (id 4) (at 168.91 67.31 0)
       (effects (font (size 1.27 1.27)) hide)
     )
@@
       (effects (font (size 1.27 1.27)) hide)
     )
+    (property "Order Number" "Farnell: 2057387" (id 4) (at 300.99 91.44 0)
+      (effects (font (size 1.27 1.27)) hide)
+    )
     (pin "2")
     (pin "3")
@@
       (effects (font (size 1.27 1.27)) hide)
     )
+    (property "Order Number" "DigiKey: 1253-1120-1-ND" (id 4) (at 157.48 60.96 0)
+      (effects (font (size 1.27 1.27)) hide)
+    )
     (pin "1")
     (pin "2")
@@
       (effects (font (size 1.27 1.27)) (justify left bottom) hide)
     )
+    (property "Order Number" "Mouser: 78-VOH1016AB-T" (id 7) (at 330.2 87.63 0)
+      (effects (font (size 1.27 1.27)) hide)
+    )
     (pin "1")
     (pin "2")
@@
       (effects (font (size 1.27 1.27)) (justify left bottom) hide)
     )
+    (property "Order Number" "Mouser: 78-VOH1016AB-T" (id 7) (at 330.2 110.49 0)
+      (effects (font (size 1.27 1.27)) hide)
+    )
     (pin "1")
     (pin "2")
@@
       (effects (font (size 1.27 1.27)) hide)
     )
+    (property "Order Number" "Farnell: 2057387" (id 4) (at 328.93 49.53 0)
+      (effects (font (size 1.27 1.27)) hide)
+    )
     (pin "2")
     (pin "3")
@@
     )
     (property "Datasheet" "http://www.ti.com/lit/sg/scyt129e/scyt129e.pdf" (id 3) (at 341.63 31.75 0)
+      (effects (font (size 1.27 1.27)) hide)
+    )
+    (property "Order Number" "Farnell: 3119379" (id 4) (at 341.63 31.75 0)
       (effects (font (size 1.27 1.27)) hide)
     )
@@
       (effects (font (size 1.27 1.27)) (justify left bottom) hide)
     )
+    (property "Order Number" "Mouser: 78-VOH1016AB-T" (id 7) (at 330.2 148.59 0)
+      (effects (font (size 1.27 1.27)) hide)
+    )
     (pin "1")
     (pin "2")
@@
       (effects (font (size 1.27 1.27)) (justify left bottom) hide)
     )
+    (property "Order Number" "Mouser: 78-VOH1016AB-T" (id 7) (at 330.2 171.45 0)
+      (effects (font (size 1.27 1.27)) hide)
+    )
     (pin "1")
     (pin "2")
@@
       (effects (font (size 1.27 1.27)) hide)
     )
+    (property "Order Number" "Farnell: 2057387" (id 4) (at 300.99 152.4 0)
+      (effects (font (size 1.27 1.27)) hide)
+    )
     (pin "2")
     (pin "3")
@@
       (effects (font (size 1.27 1.27)) (justify left bottom) hide)
     )
+    (property "Order Number" "Mouser: 78-VOH1016AB-T" (id 7) (at 330.2 208.28 0)
+      (effects (font (size 1.27 1.27)) hide)
+    )
     (pin "1")
     (pin "2")
@@
       (effects (font (size 1.27 1.27)) (justify left bottom) hide)
     )
+    (property "Order Number" "Mouser: 78-VOH1016AB-T" (id 7) (at 330.2 231.14 0)
+      (effects (font (size 1.27 1.27)) hide)
+    )
     (pin "1")
     (pin "2")
@@
       (effects (font (size 1.27 1.27)) hide)
     )
+    (property "Order Number" "Farnell: 2057387" (id 4) (at 300.99 212.09 0)
+      (effects (font (size 1.27 1.27)) hide)
+    )
     (pin "2")
     (pin "3")
@@
     )
     (property "Datasheet" "~" (id 3) (at 113.03 220.98 0)
+      (effects (font (size 1.27 1.27)) hide)
+    )
+    (property "Order Number" "Farnell: 1833843" (id 4) (at 113.03 220.98 0)
       (effects (font (size 1.27 1.27)) hide)
     )
@@
       (effects (font (size 1.27 1.27)) hide)
     )
+    (property "Order Number" "Farnell: 3122539" (id 4) (at 87.63 214.63 0)
+      (effects (font (size 1.27 1.27)) hide)
+    )
     (pin "1")
     (pin "2")
@@
       (effects (font (size 1.27 1.27)) hide)
     )
+    (property "Order Number" "Farnell: 1833843" (id 4) (at 66.04 220.98 0)
+      (effects (font (size 1.27 1.27)) hide)
+    )
